File: KiCad_Designs/Prototype_design/prueba_1.sch (KiCad schematic (older format))
At the start: 89 parts, among them J1 AIN_2, J10 External Clk, J11 M2, J12 Mode_Selection, J13 Alimentacion, J2 AIN_1, J3 AIN_3, J4 AIN_2W, J5 AIN_1W, J6 AIN_3W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

Commit message: Prototype Schematic Updated
Parts:
- removed J10: External Clk, Connector_PinHeader_2.54mm:PinHeader_1x02_P2.54mm_Vertical, symbol Connector:Conn_01x02_Male
Other:
- note added: "Diseño por Jorge Rafael Paredes Dubón, basado en la tarjeta de desarollo del ADS131A04"
- moved on the sheet: C1, C10, C11, C12, C13, C14, C15, C16, C17, C18, C19, C2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
